File: hardware/kicad/konservasi_air.kicad_sch (KiCad schematic)
At the start: 7 parts, among them J1 ADS1115, J2 DS18B20, J3 TDS, J4 TURBIDITY, J5 pH, J6 SERVO, U1 ESP32-DevKitC

Commit message: Update Schematics
Parts:
- added C1, C2: 100n, Capacitor_THT:C_Disc_D7.5mm_W5.0mm_P7.50mm, symbol Device:C_Small
- added C3, C4: 47u, Capacitor_THT:C_Radial_D5.0mm_H11.0mm_P2.00mm, symbol Device:C_Polarized_Small
- added D1: Red, LED_THT:LED_D3.0mm, symbol Device:LED_Small
- added D2: IN4004, Diode_THT:D_A-405_P12.70mm_Horizontal, symbol Device:D_Small
- added J10: PUMP, Connector_PinSocket_2.54mm:PinSocket_1x02_P2.54mm_Vertical, symbol Connector_Generic:Conn_01x02
- added J11: DC_IN_TERMINAL, TerminalBlock_Phoenix:TerminalBlock_Phoenix_MPT-0,5-2-2.54_1x02_P2.54mm_Horizontal, symbol Connector:Screw_Terminal_01x02
- added J7: OLED, Connector_Molex:Molex_SL_171971-0004_1x04_P2.54mm_Vertical, symbol Connector_Generic:Conn_01x04
- added J8: ADS1115_ADDR_JP, Connector_PinHeader_2.54mm:PinHeader_2x04_P2.54mm_Vertical, symbol Connector_Generic:Conn_02x04_Top_Bottom
- added J9: DC_IN_JACK, Connector_BarrelJack:BarrelJack_Horizontal, symbol Connector:Screw_Terminal_01x02
- added Q1: IRF520, Package_TO_SOT_THT:TO-220-3_Vertical, symbol Transistor_FET:IRF540N
- added R1, R3, R4: 4.7k, Resistor_THT:R_Axial_DIN0309_L9.0mm_D3.2mm_P12.70mm_Horizontal, symbol Device:R_Small
- added R2: 1.5k, Resistor_THT:R_Axial_DIN0309_L9.0mm_D3.2mm_P12.70mm_Horizontal, symbol Device:R_Small
- added R5: 1k, Resistor_THT:R_Axial_DIN0309_L9.0mm_D3.2mm_P12.70mm_Horizontal, symbol Device:R_Small
- added SW1: ESP_EN, Button_Switch_THT:SW_PUSH_6mm, symbol Switch:SW_Push
- added SW2: ESP_EN_JP, Connector_PinSocket_2.54mm:PinSocket_1x02_P2.54mm_Vertical, symbol Switch:SW_Push
- J1: footprint (none) -> Connector_PinSocket_2.54mm:PinSocket_1x10_P2.54mm_Vertical
- J2, J3, J4, J6: footprint (none) -> Connector_Molex:Molex_SL_171971-0003_1x03_P2.54mm_Vertical
- J5: footprint (none) -> Connector_Molex:Molex_SL_171971-0006_1x06_P2.54mm_Vertical
Connections:
- net +3V3: now also C1.1
- net +5V: now also C2.1, C3.1, C4.1, D2.1 (K), J10.1 (Pin_1), J11.1 (Pin_1), J7.1 (Pin_1), J8.6 (Pin_6), J9.1 (Pin_1), R2.2, R3.2, R4.2
- net ADS1115_ADDR: now also J8.1 (Pin_1), J8.2 (Pin_2), J8.3 (Pin_3), J8.4 (Pin_4)
- net ADS1115_SCL: now also J7.3 (Pin_3), J8.8 (Pin_8), R3.1
- net ADS1115_SDA: now also J7.4 (Pin_4), J8.7 (Pin_7), R4.1
- net DS18B20_DIGITAL: now also R1.2
- net GND: now also C1.2, C2.2, C3.2, C4.2, D1.1 (K), J11.2 (Pin_2), J7.2 (Pin_2), J8.5 (Pin_5), J9.2 (Pin_2), Q1.3 (S), SW1.1, SW2.1
- net SERVO_PWM: now also U1.31 (GPIO19)
- net at U1.2 (CHIP_PU): now also SW1.2, SW2.2
- net at U1.37 (GPIO23): now also R1.1
- new net: Q1.1 (G), R5.1
- new net: D1.2 (A), R2.1
- new net PUMP_DIGITAL: R5.2
- new net PUMP_GND: D2.2 (A), J10.2 (Pin_2), Q1.2 (D)
Other:
- note added: "0X48 0X49 0X4A 0X4B"
- note added: "ADS1115"
- note added: "ESP32 DEV. MODULE"
- note added: "I2C ADDRESS"
- note added: "SENSORS"
- note added: "WATER PUMP (OUT)"
- moved on the sheet: J1, J2, J3, J4, J5, J6, U1

Commit message: PCB Layout Update
Parts:
- removed J8: ADS1115_ADDR_JP, Connector_PinHeader_2.54mm:PinHeader_2x04_P2.54mm_Vertical, symbol Connector_Generic:Conn_02x04_Top_Bottom
- removed SW1: ESP_EN, Button_Switch_THT:SW_PUSH_6mm, symbol Switch:SW_Push
- added J8: ADS1115_ADDR, Connector_PinHeader_2.54mm:PinHeader_2x04_P2.54mm_Vertical, symbol Connector_Generic:Conn_02x04_Odd_Even
- C1, C2: footprint Capacitor_THT:C_Disc_D7.5mm_W5.0mm_P7.50mm -> Capacitor_THT:C_Disc_D5.0mm_W2.5mm_P5.00mm
- D2: footprint Diode_THT:D_A-405_P12.70mm_Horizontal -> Diode_THT:D_DO-34_SOD68_P7.62mm_Horizontal
- J10: footprint Connector_PinSocket_2.54mm:PinSocket_1x02_P2.54mm_Vertical -> Connector_Molex:Molex_SL_171971-0002_1x02_P2.54mm_Vertical
- R1, R2, R3, R4, R5: footprint Resistor_THT:R_Axial_DIN0309_L9.0mm_D3.2mm_P12.70mm_Horizontal -> Resistor_THT:R_Axial_DIN0204_L3.6mm_D1.6mm_P7.62mm_Horizontal
- SW1: renamed from SW2; footprint Connector_PinSocket_2.54mm:PinSocket_1x02_P2.54mm_Vertical -> Connector_Molex:Molex_SL_171971-0002_1x02_P2.54mm_Vertical
Connections:
- net +5V: now also J8.4 (Pin_4)
- net ADS1115_ADDR: now also J8.1 (Pin_1), J8.3 (Pin_3), J8.5 (Pin_5), J8.7 (Pin_7)
- net ADS1115_SCL: now also J8.8 (Pin_8)
- net ADS1115_SDA: now also J8.6 (Pin_6)
- net GND: now also J8.2 (Pin_2)
Other:
- moved on the sheet: SW1
Changed lines of the file:
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@@
   (junction (at 140.97 64.77) (diameter 0) (color 0 0 0 0)
   )
-  (junction (at 44.45 41.91) (diameter 0) (color 0 0 0 0)
-  )
   (junction (at 34.29 189.23) (diameter 0) (color 0 0 0 0)
   )
@@
     (stroke (width 0) (type default))
   )
-  (wire (pts (xy 29.21 41.91) (xy 44.45 41.91))
-    (stroke (width 0) (type default))
-  )
   (wire (pts (xy 39.37 143.51) (xy 52.07 143.51))
     (stroke (width 0) (type default))
@@
     (stroke (width 0) (type default))
   )
+  (wire (pts (xy 44.45 30.48) (xy 44.45 31.75))
+    (stroke (width 0) (type default))
+  )
   (wire (pts (xy 146.05 137.16) (xy 161.29 137.16))
     (stroke (width 0) (type default))
@@
   )
   (wire (pts (xy 62.23 189.23) (xy 48.26 189.23))
+    (stroke (width 0) (type default))
+  )
+  (wire (pts (xy 44.45 41.91) (xy 44.45 40.64))
     (stroke (width 0) (type default))
   )
@@
         (path "/b0a95a89-a5ca-444f-aff6-2e93a9826d99"
           (reference "#PWR016") (unit 1)
-        )
-      )
-    )
-  )
-  (symbol (lib_id "Switch:SW_Push") (at 29.21 36.83 270) (unit 1)
-    (in_bom yes) (on_board yes) (dnp no)
-    (property "Reference" "SW1" (at 27.94 38.1 90)
-      (effects (font (size 1.27 1.27)) (justify right))
-    )
-    (property "Value" "ESP_EN" (at 27.94 35.56 90)
-      (effects (font (size 1.27 1.27)) (justify right))
-    )
-    (property "Footprint" "Button_Switch_THT:SW_PUSH_6mm" (at 34.29 36.83 0)
-      (effects (font (size 1.27 1.27)) hide)
-    )
-    (property "Datasheet" "~" (at 34.29 36.83 0)
-      (effects (font (size 1.27 1.27)) hide)
-    )
-    (pin "1")
-    (pin "2")
-    (instances
-      (project "konservasi_air"
-        (path "/b0a95a89-a5ca-444f-aff6-2e93a9826d99"
-          (reference "SW1") (unit 1)
         )
       )
@@
       (effects (font (size 1.27 1.27)) (justify right))
     )
-    (property "Footprint" "Resistor_THT:R_Axial_DIN0309_L9.0mm_D3.2mm_P12.70mm_Horizontal" (at 137.16 58.42 0)
+    (property "Footprint" "Resistor_THT:R_Axial_DIN0204_L3.6mm_D1.6mm_P7.62mm_Horizontal" (at 137.16 58.42 0)
       (effects (font (size 1.27 1.27)) hide)
     )
@@
         (path "/b0a95a89-a5ca-444f-aff6-2e93a9826d99"
           (reference "C3") (unit 1)
+        )
+      )
+    )
+  )
+  (symbol (lib_id "Connector_Generic:Conn_02x04_Odd_Even") (at 40.64 186.69 0) (unit 1)
+    (in_bom yes) (on_board yes) (dnp no) (fields_autoplaced)
+    (property "Reference" "J8" (at 41.91 177.8 0)
+      (effects (font (size 1.27 1.27)))
+    )
+    (property "Value" "ADS1115_ADDR" (at 41.91 180.34 0)
+      (effects (font (size 1.27 1.27)))
+    )
+    (property "Footprint" "Connector_PinHeader_2.54mm:PinHeader_2x04_P2.54mm_Vertical" (at 40.64 186.69 0)
+      (effects (font (size 1.27 1.27)) hide)
+    )
+    (property "Datasheet" "~" (at 40.64 186.69 0)
+      (effects (font (size 1.27 1.27)) hide)
+    )
+    (pin "1")
+    (pin "2")
+    (pin "3")
+    (pin "4")
+    (pin "5")
+    (pin "6")
+    (pin "7")
+    (pin "8")
+    (instances
+      (project "konservasi_air"
+        (path "/b0a95a89-a5ca-444f-aff6-2e93a9826d99"
+          (reference "J8") (unit 1)
         )
       )
@@
       (effects (font (size 1.27 1.27)))
     )
-    (property "Footprint" "Resistor_THT:R_Axial_DIN0309_L9.0mm_D3.2mm_P12.70mm_Horizontal" (at 163.83 137.16 0)
+    (property "Footprint" "Resistor_THT:R_Axial_DIN0204_L3.6mm_D1.6mm_P7.62mm_Horizontal" (at 163.83 137.16 0)
       (effects (font (size 1.27 1.27)) hide)
     )
@@
       (effects (font (size 1.27 1.27)) (justify left))
     )
-    (property "Footprint" "Capacitor_THT:C_Disc_D7.5mm_W5.0mm_P7.50mm" (at 87.63 29.21 0)
+    (property "Footprint" "Capacitor_THT:C_Disc_D5.0mm_W2.5mm_P5.00mm" (at 87.63 29.21 0)
       (effects (font (size 1.27 1.27)) hide)
     )
@@
     )
   )
-  (symbol (lib_id "Switch:SW_Push") (at 44.45 36.83 270) (unit 1)
+  (symbol (lib_id "Switch:SW_Push") (at 44.45 35.56 270) (unit 1)
     (in_bom yes) (on_board yes) (dnp no)
-    (property "Reference" "SW2" (at 43.18 38.1 90)
+    (property "Reference" "SW1" (at 43.18 36.83 90)
       (effects (font (size 1.27 1.27)) (justify right))
     )
-    (property "Value" "ESP_EN_JP" (at 43.18 35.56 90)
+    (property "Value" "ESP_EN_JP" (at 43.18 34.29 90)
       (effects (font (size 1.27 1.27)) (justify right))
     )
-    (property "Footprint" "Connector_PinSocket_2.54mm:PinSocket_1x02_P2.54mm_Vertical" (at 49.53 36.83 0)
-      (effects (font (size 1.27 1.27)) hide)
-    )
-    (property "Datasheet" "~" (at 49.53 36.83 0)
-      (effects (font (size 1.27 1.27)) hide)
-    )
-    (pin "1")
-    (pin "2")
-    (instances
-      (project "konservasi_air"
-        (path "/b0a95a89-a5ca-444f-aff6-2e93a9826d99"
-          (reference "SW2") (unit 1)
+    (property "Footprint" "Connector_Molex:Molex_SL_171971-0002_1x02_P2.54mm_Vertical" (at 49.53 35.56 0)
+      (effects (font (size 1.27 1.27)) hide)
+    )
+    (property "Datasheet" "~" (at 49.53 35.56 0)
+      (effects (font (size 1.27 1.27)) hide)
+    )
+    (pin "1")
+    (pin "2")
+    (instances
+      (project "konservasi_air"
+        (path "/b0a95a89-a5ca-444f-aff6-2e93a9826d99"
+          (reference "SW1") (unit 1)
         )
       )
@@
       (effects (font (size 1.27 1.27)))
     )
-    (property "Footprint" "Resistor_THT:R_Axial_DIN0309_L9.0mm_D3.2mm_P12.70mm_Horizontal" (at 273.05 60.96 0)
+    (property "Footprint" "Resistor_THT:R_Axial_DIN0204_L3.6mm_D1.6mm_P7.62mm_Horizontal" (at 273.05 60.96 0)
       (effects (font (size 1.27 1.27)) hide)
     )
@@
       (effects (font (size 1.27 1.27)) (justify right))
     )
-    (property "Footprint" "Diode_THT:D_A-405_P12.70mm_Horizontal" (at 208.28 140.97 90)
+    (property "Footprint" "Diode_THT:D_DO-34_SOD68_P7.62mm_Horizontal" (at 208.28 140.97 90)
       (effects (font (size 1.27 1.27)) hide)
     )
@@
         (path "/b0a95a89-a5ca-444f-aff6-2e93a9826d99"
           (reference "D2") (unit 1)
-        )
-      )
-    )
-  )
-  (symbol (lib_id "power:GND") (at 29.21 31.75 180) (unit 1)
-    (in_bom yes) (on_board yes) (dnp no) (fields_autoplaced)
-    (property "Reference" "#PWR018" (at 29.21 25.4 0)
-      (effects (font (size 1.27 1.27)) hide)
-    )
-    (property "Value" "GND" (at 29.21 26.67 0)
-      (effects (font (size 1.27 1.27)))
-    )
-    (property "Footprint" "" (at 29.21 31.75 0)
-      (effects (font (size 1.27 1.27)) hide)
-    )
-    (property "Datasheet" "" (at 29.21 31.75 0)
-      (effects (font (size 1.27 1.27)) hide)
-    )
-    (pin "1")
-    (instances
-      (project "konservasi_air"
-        (path "/b0a95a89-a5ca-444f-aff6-2e93a9826d99"
-          (reference "#PWR018") (unit 1)
         )
       )
@@
       (effects (font (size 1.27 1.27)))
     )
-    (property "Footprint" "Resistor_THT:R_Axial_DIN0309_L9.0mm_D3.2mm_P12.70mm_Horizontal" (at 125.73 69.85 0)
+    (property "Footprint" "Resistor_THT:R_Axial_DIN0204_L3.6mm_D1.6mm_P7.62mm_Horizontal" (at 125.73 69.85 0)
       (effects (font (size 1.27 1.27)) hide)
     )
@@
       (effects (font (size 1.27 1.27)) (justify right))
     )
-    (property "Footprint" "Resistor_THT:R_Axial_DIN0309_L9.0mm_D3.2mm_P12.70mm_Horizontal" (at 140.97 58.42 0)
+    (property "Footprint" "Resistor_THT:R_Axial_DIN0204_L3.6mm_D1.6mm_P7.62mm_Horizontal" (at 140.97 58.42 0)
       (effects (font (size 1.27 1.27)) hide)
     )
@@
       (effects (font (size 1.27 1.27)) (justify left))
     )
-    (property "Footprint" "Capacitor_THT:C_Disc_D7.5mm_W5.0mm_P7.50mm" (at 74.93 29.21 0)
+    (property "Footprint" "Capacitor_THT:C_Disc_D5.0mm_W2.5mm_P5.00mm" (at 74.93 29.21 0)
       (effects (font (size 1.27 1.27)) hide)
     )
@@
       (effects (font (size 1.27 1.27)) (justify left))
     )
-    (property "Footprint" "Connector_PinSocket_2.54mm:PinSocket_1x02_P2.54mm_Vertical" (at 219.71 139.7 0)
+    (property "Footprint" "Connector_Molex:Molex_SL_171971-0002_1x02_P2.54mm_Vertical" (at 219.71 139.7 0)
       (effects (font (size 1.27 1.27)) hide)
     )
@@
         )
       )
-    )
-  )
-  (symbol (lib_id "Connector_Generic:Conn_02x04_Top_Bottom") (at 40.64 186.69 0) (unit 1)
-    (in_bom yes) (on_board yes) (dnp no) (fields_autoplaced)
-    (property "Reference" "J8" (at 41.91 177.8 0)
-      (effects (font (size 1.27 1.27)))
-    )
-    (property "Value" "ADS1115_ADDR_JP" (at 41.91 180.34 0)
-      (effects (font (size 1.27 1.27)))
-    )
-    (property "Footprint" "Connector_PinHeader_2.54mm:PinHeader_2x04_P2.54mm_Vertical" (at 40.64 186.69 0)
-      (effects (font (size 1.27 1.27)) hide)
-    )
-    (property "Datasheet" "~" (at 40.64 186.69 0)
-      (effects (font (size 1.27 1.27)) hide)
-    )
-    (pin "1")
-    (pin "2")
-    (pin "3")
-    (pin "4")
-    (pin "5")
-    (pin "6")
-    (pin "7")
-    (pin "8")
-    (instances
-      (project "konservasi_air"
-        (path "/b0a95a89-a5ca-444f-aff6-2e93a9826d99"
-          (reference "J8") (unit 1)
-        )
-      )

Commit message: PCB Update
Parts:
- added J12: ESP_GPIO_LEFT, Connector_PinHeader_2.54mm:PinHeader_1x19_P2.54mm_Vertical, symbol Connector_Generic:Conn_01x19
- added J13: ESP_GPIO_RIGHT, Connector_PinHeader_2.54mm:PinHeader_1x19_P2.54mm_Vertical, symbol Connector_Generic:Conn_01x19
Connections:
- net +3V3: now also J12.1 (Pin_1)
- net +5V: now also J12.19 (Pin_19)
- net ADS1115_SCL: now also J13.3 (Pin_3)
- net ADS1115_SDA: now also J13.6 (Pin_6)
- net GND: now also J12.14 (Pin_14), J13.1 (Pin_1), J13.7 (Pin_7)
- net PUMP_DIGITAL: now also U1.13 (MTDI/GPIO12/ADC2_CH5), J12.13 (Pin_13)
- net SERVO_PWM: now also J13.8 (Pin_8)
- net ESP_GPIO26: now reaches U1.10 (DAC_2/ADC2_CH9/GPIO26)
- net ESP_GPIO26: now also J12.10 (Pin_10)
- net ESP_GPIO27: now reaches U1.11 (ADC2_CH7/GPIO27)
- net ESP_GPIO27: now also J12.11 (Pin_11)
- net ESP_GPIO14: now reaches U1.12 (MTMS/GPIO14/ADC2_CH6)
- net ESP_GPIO14: now also J12.12 (Pin_12)
- net ESP_GPIO13: now reaches U1.15 (MTCK/GPIO13/ADC2_CH4)
- net ESP_GPIO13: now also J12.15 (Pin_15)
- net ESP_GPIO09: now reaches U1.16 (SD_DATA2/GPIO9)
- net ESP_GPIO09: now also J12.16 (Pin_16)
- net ESP_GPIO10: now reaches U1.17 (SD_DATA3/GPIO10)
- net ESP_GPIO10: now also J12.17 (Pin_17)
- net ESP_CMD: now reaches U1.18 (CMD)
- net ESP_CMD: now also J12.18 (Pin_18)
- net ESP_RESET: now reaches SW1.2, U1.2 (CHIP_PU)
- net ESP_RESET: now also J12.2 (Pin_2)
- net ESP_GPIO06: now reaches U1.20 (SD_CLK/GPIO6)
- net ESP_GPIO06: now also J13.19 (Pin_19)
- net ESP_GPIO07: now reaches U1.21 (SD_DATA0/GPIO7)
- net ESP_GPIO07: now also J13.18 (Pin_18)
- net ESP_GPIO08: now reaches U1.22 (SD_DATA1/GPIO8)
- net ESP_GPIO08: now also J13.17 (Pin_17)
- net ESP_GPIO15: now reaches U1.23 (MTDO/GPIO15/ADC2_CH3)
- net ESP_GPIO15: now also J13.16 (Pin_16)
- net ESP_GPIO02: now reaches U1.24 (ADC2_CH2/GPIO2)
- net ESP_GPIO02: now also J13.15 (Pin_15)
- net ESP_GPIO00: now reaches U1.25 (GPIO0/BOOT/ADC2_CH1)
- net ESP_GPIO00: now also J13.14 (Pin_14)
- net ESP_GPIO04: now reaches U1.26 (ADC2_CH0/GPIO4)
- net ESP_GPIO04: now also J13.13 (Pin_13)
- net ESP_GPIO16: now reaches U1.27 (GPIO16)
- net ESP_GPIO16: now also J13.12 (Pin_12)
- net ESP_GPIO17: now reaches U1.28 (GPIO17)
- net ESP_GPIO17: now also J13.11 (Pin_11)
- net ESP_GPIO05: now reaches U1.29 (GPIO5)
- net ESP_GPIO05: now also J13.10 (Pin_10)
- net ESP_GPIO36: now reaches U1.3 (SENSOR_VP/GPIO36/ADC1_CH0)
- net ESP_GPIO36: now also J12.3 (Pin_3)
- net ESP_GPIO18: now reaches U1.30 (GPIO18)
- net ESP_GPIO18: now also J13.9 (Pin_9)
- net ESP_GPIO03: now reaches U1.34 (U0RXD/GPIO3)
- net ESP_GPIO03: now also J13.5 (Pin_5)
- net ESP_GPIO01: now reaches U1.35 (U0TXD/GPIO1)
- net ESP_GPIO01: now also J13.4 (Pin_4)
- net ESP_GPIO23: now reaches R1.1, U1.37 (GPIO23)
- net ESP_GPIO23: now also J13.2 (Pin_2)
- net ESP_GPIO39: now reaches U1.4 (SENSOR_VN/GPIO39/ADC1_CH3)
- net ESP_GPIO39: now also J12.4 (Pin_4)
- net ESP_GPIO34: now reaches U1.5 (VDET_1/GPIO34/ADC1_CH6)
- net ESP_GPIO34: now also J12.5 (Pin_5)
- net ESP_GPIO35: now reaches U1.6 (VDET_2/GPIO35/ADC1_CH7)
- net ESP_GPIO35: now also J12.6 (Pin_6)
- net ESP_GPIO32: now reaches U1.7 (32K_XP/GPIO32/ADC1_CH4)
- net ESP_GPIO32: now also J12.7 (Pin_7)
- net ESP_GPIO33: now reaches U1.8 (32K_XN/GPIO33/ADC1_CH5)
- net ESP_GPIO33: now also J12.8 (Pin_8)
- net ESP_GPIO25: now reaches U1.9 (DAC_1/ADC2_CH8/GPIO25)
- net ESP_GPIO25: now also J12.9 (Pin_9)
Other:
- moved on the sheet: C1, C2, C3, C4, D1, J11, J9, R1, R2, R3, R4, SW1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

Commit message: Done Routing
Parts:
- removed J8: ADS1115_ADDR, Connector_PinHeader_2.54mm:PinHeader_2x04_P2.54mm_Vertical, symbol Connector_Generic:Conn_02x04_Odd_Even
- removed J9: DC_IN_JACK, Connector_BarrelJack:BarrelJack_Horizontal, symbol Connector:Screw_Terminal_01x02
- added J9: Barrel_Jack_Switch, Connector_BarrelJack:BarrelJack_Horizontal, symbol Connector:Barrel_Jack_Switch
- added JP1: ADS1115_ADDR_5V, Jumper:SolderJumper-2_P1.3mm_Open_RoundedPad1.0x1.5mm, symbol Jumper:SolderJumper_2_Open
- added JP2: ADS1115_ADDR_SDA, Jumper:SolderJumper-2_P1.3mm_Open_RoundedPad1.0x1.5mm, symbol Jumper:SolderJumper_2_Open
- added JP3: ADS1115_ADDR_SCL, Jumper:SolderJumper-2_P1.3mm_Open_RoundedPad1.0x1.5mm, symbol Jumper:SolderJumper_2_Open
Connections:
- net +5V: now also J9.1, JP1.2 (B)
- net ADS1115_ADDR: now also JP1.1 (A), JP2.1 (A), JP3.1 (A)
- net ADS1115_SCL: now also J7.4 (Pin_4), JP3.2 (B); no longer J7.3 (Pin_3)
- net ADS1115_SDA: now also J7.3 (Pin_3), JP2.2 (B); no longer J7.4 (Pin_4)
- net ESP_GPIO25: now also J6.1 (Pin_1)
- net GND: now also J9.2
- net SERVO_PWM renamed ESP_GPIO19
- net ESP_GPIO19: no longer J6.1 (Pin_1)
- no-connect marks 0 -> 1
Other:
- note added: "0X48 (Default) 0X49 0X4A 0X4B"
- note removed: "0X48 0X49 0X4A 0X4B"
